Commit message: working sim with thermal

File: simulation/husky_config/husky_custom_description/urdf/husky.urdf.xacro (robot description, xacro)
@@ -70,5 +70,5 @@
         <origin xyz="0 0 0" rpy="1.57079632679 0 0" />
         <geometry>
-          <mesh filename="$(find mbzirc_husky)/models/box.dae" scale="1 1 1" />
+          <mesh filename="$(find mbzirc_husky)/models/bluefox.dae" scale="1 1 1" />
         </geometry>
       </visual>
@@ -136,7 +136,7 @@
     image_width="32"
     image_height="32"
-    x="0.13"
+    x="0.4"
     y="0"
-    z="2.185"
+    z="0.4"
     roll="0"
     pitch="0.0"
