Commit message: sim files, bounds config

File: sensor_control/simulation/gazebo/husky_config/husky_custom_description/urdf/husky.urdf.xacro (robot description, xacro)
@@ -2,6 +2,6 @@
 <robot xmlns:xacro="http://www.ros.org/wiki/xacro" name="example">
   <xacro:include filename="$(find velodyne_description)/urdf/VLP-16.urdf.xacro"/>
-  <VLP-16 parent="top_plate_link" name="velodyne" topic="/velodyne_points" hz="10" samples="440">
-     <origin xyz="-0.075 0.0 0.08635" rpy="0 0 0" />
+  <VLP-16 parent="base_link" name="velodyne" topic="/velodyne_points" hz="10" samples="440">
+     <origin xyz="-0.075 0.0 0.4" rpy="0 0 0" />
   </VLP-16>
   <!-- Macro to add a thermal camera {-->
